File: sec.kicad_sch (KiCad schematic)
At the start: 6 parts, among them U3 4081, U4 4510, U5 4510

Commit message: Asigning footprints
Parts:
- C5, C6, C7: footprint (none) -> Capacitor_SMD:C_0603_1608Metric_Pad1.08x0.95mm_HandSolder; LCSC Part (none) -> C2170999
- U3: LCSC Part (none) -> C5145433
- U3: footprint Package_DIP:DIP-14_W7.62mm_Socket_LongPads -> (none); LCSC Part (none) -> C5145433
- U4, U5: footprint (none) -> Package_SO:TSSOP-16_4.4x5mm_P0.65mm; LCSC Part (none) -> C2862976
Changed lines of the file:
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@@
 			)
 		)
-		(property "Footprint" ""
+		(property "Footprint" "Capacitor_SMD:C_0603_1608Metric_Pad1.08x0.95mm_HandSolder"
 			(at 85.09 58.7248 0)
 			(hide yes)
@@
 			)
 		)
+		(property "LCSC Part" "C2170999"
+			(at 81.28 59.69 90)
+			(hide yes)
+			(show_name no)
+			(do_not_autoplace no)
+			(effects
+				(font
+					(size 1.27 1.27)
+				)
+			)
+		)
 		(pin "1"
 		)
@@
 			)
 		)
-		(property "Footprint" ""
+		(property "Footprint" "Capacitor_SMD:C_0603_1608Metric_Pad1.08x0.95mm_HandSolder"
 			(at 50.8 157.7848 0)
 			(hide yes)
@@
 		(property "Description" "Unpolarized capacitor"
 			(at 46.99 158.75 0)
+			(hide yes)
+			(show_name no)
+			(do_not_autoplace no)
+			(effects
+				(font
+					(size 1.27 1.27)
+				)
+			)
+		)
+		(property "LCSC Part" "C2170999"
+			(at 46.99 158.75 90)
 			(hide yes)
 			(show_name no)
@@
 			)
 		)
+		(property "LCSC Part" "C5145433"
+			(at 218.44 63.5 0)
+			(hide yes)
+			(show_name no)
+			(do_not_autoplace no)
+			(effects
+				(font
+					(size 1.27 1.27)
+				)
+			)
+		)
 		(pin "4"
 		)
@@
 			)
 		)
-		(property "Footprint" ""
+		(property "Footprint" "Package_SO:TSSOP-16_4.4x5mm_P0.65mm"
 			(at 179.07 71.12 0)
 			(hide yes)
@@
 			)
 		)
+		(property "LCSC Part" "C2862976"
+			(at 179.07 71.12 0)
+			(hide yes)
+			(show_name no)
+			(do_not_autoplace no)
+			(effects
+				(font
+					(size 1.27 1.27)
+				)
+			)
+		)
 		(pin "12"
 		)
@@
 			)
 		)
-		(property "Footprint" ""
+		(property "Footprint" "Package_SO:TSSOP-16_4.4x5mm_P0.65mm"
 			(at 85.09 80.01 0)
 			(hide yes)
@@
 			)
 		)
+		(property "LCSC Part" "C2862976"
+			(at 85.09 80.01 0)
+			(hide yes)
+			(show_name no)
+			(do_not_autoplace no)
+			(effects
+				(font
+					(size 1.27 1.27)
+				)
+			)
+		)
 		(pin "12"
 		)
@@
 			)
 		)
-		(property "Footprint" "Package_DIP:DIP-14_W7.62mm_Socket_LongPads"
+		(property "Footprint" ""
 			(at 124.46 74.93 0)
 			(hide yes)
@@
 		)
 		(property "Description" "Quad And 2 inputs"
+			(at 124.46 74.93 0)
+			(hide yes)
+			(show_name no)
+			(do_not_autoplace no)
+			(effects
+				(font
+					(size 1.27 1.27)
+				)
+			)
+		)
+		(property "LCSC Part" "C5145433"
 			(at 124.46 74.93 0)
 			(hide yes)
@@
 			)
 		)
+		(property "LCSC Part" "C5145433"
+			(at 50.8 173.99 0)
+			(hide yes)
+			(show_name no)
+			(do_not_autoplace no)
+			(effects
+				(font
+					(size 1.27 1.27)
+				)
+			)
+		)
 		(pin "4"
 		)
@@
 			)
 		)
-		(property "Footprint" ""
+		(property "Footprint" "Capacitor_SMD:C_0603_1608Metric_Pad1.08x0.95mm_HandSolder"
 			(at 179.07 49.8348 0)
 			(hide yes)
@@
 			(hide yes)
 			(show_name no)
+			(do_not_autoplace no)
+			(effects
+				(font
+					(size 1.27 1.27)
+				)
+			)
+		)
+		(property "LCSC Part" "C2170999"
+			(at 175.26 50.8 90)
+			(hide yes)
+			(show_name no)

Commit message: Asigning footprints
Parts:
- C5, C6, C7: footprint Capacitor_SMD:C_0603_1608Metric_Pad1.08x0.95mm_HandSolder -> Capacitor_SMD:C_0603_1608Metric; LCSC Part C2170999 -> (none)
- U3: LCSC Part C5145433 -> (none)
- U4, U5: footprint Package_SO:TSSOP-16_4.4x5mm_P0.65mm -> (none); LCSC Part C2862976 -> (none)
Changed lines of the file:
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@@
 			)
 		)
-		(property "Footprint" "Capacitor_SMD:C_0603_1608Metric_Pad1.08x0.95mm_HandSolder"
+		(property "Footprint" "Capacitor_SMD:C_0603_1608Metric"
 			(at 85.09 58.7248 0)
 			(hide yes)
@@
 			)
 		)
-		(property "LCSC Part" "C2170999"
-			(at 81.28 59.69 90)
-			(hide yes)
-			(show_name no)
-			(do_not_autoplace no)
-			(effects
-				(font
-					(size 1.27 1.27)
-				)
-			)
-		)
 		(pin "1"
 		)
@@
 			)
 		)
-		(property "Footprint" "Capacitor_SMD:C_0603_1608Metric_Pad1.08x0.95mm_HandSolder"
+		(property "Footprint" "Capacitor_SMD:C_0603_1608Metric"
 			(at 50.8 157.7848 0)
 			(hide yes)
@@
 		(property "Description" "Unpolarized capacitor"
 			(at 46.99 158.75 0)
-			(hide yes)
-			(show_name no)
-			(do_not_autoplace no)
-			(effects
-				(font
-					(size 1.27 1.27)
-				)
-			)
-		)
-		(property "LCSC Part" "C2170999"
-			(at 46.99 158.75 90)
 			(hide yes)
 			(show_name no)
@@
 			)
 		)
-		(property "LCSC Part" "C5145433"
-			(at 218.44 63.5 0)
-			(hide yes)
-			(show_name no)
-			(do_not_autoplace no)
-			(effects
-				(font
-					(size 1.27 1.27)
-				)
-			)
-		)
 		(pin "4"
 		)
@@
 			)
 		)
-		(property "Footprint" "Package_SO:TSSOP-16_4.4x5mm_P0.65mm"
+		(property "Footprint" ""
 			(at 179.07 71.12 0)
 			(hide yes)
@@
 			)
 		)
-		(property "LCSC Part" "C2862976"
-			(at 179.07 71.12 0)
-			(hide yes)
-			(show_name no)
-			(do_not_autoplace no)
-			(effects
-				(font
-					(size 1.27 1.27)
-				)
-			)
-		)
 		(pin "12"
 		)
@@
 			)
 		)
-		(property "Footprint" "Package_SO:TSSOP-16_4.4x5mm_P0.65mm"
+		(property "Footprint" ""
 			(at 85.09 80.01 0)
 			(hide yes)
@@
 			)
 		)
-		(property "LCSC Part" "C2862976"
-			(at 85.09 80.01 0)
-			(hide yes)
-			(show_name no)
-			(do_not_autoplace no)
-			(effects
-				(font
-					(size 1.27 1.27)
-				)
-			)
-		)
 		(pin "12"
 		)
@@
 		)
 		(property "Description" "Quad And 2 inputs"
-			(at 124.46 74.93 0)
-			(hide yes)
-			(show_name no)
-			(do_not_autoplace no)
-			(effects
-				(font
-					(size 1.27 1.27)
-				)
-			)
-		)
-		(property "LCSC Part" "C5145433"
 			(at 124.46 74.93 0)
 			(hide yes)
@@
 			)
 		)
-		(property "LCSC Part" "C5145433"
-			(at 50.8 173.99 0)
-			(hide yes)
-			(show_name no)
-			(do_not_autoplace no)
-			(effects
-				(font
-					(size 1.27 1.27)
-				)
-			)
-		)
 		(pin "4"
 		)
@@
 			)
 		)
-		(property "Footprint" "Capacitor_SMD:C_0603_1608Metric_Pad1.08x0.95mm_HandSolder"
+		(property "Footprint" "Capacitor_SMD:C_0603_1608Metric"
 			(at 179.07 49.8348 0)
 			(hide yes)
@@
 			(hide yes)
 			(show_name no)
-			(do_not_autoplace no)
-			(effects
-				(font
-					(size 1.27 1.27)
-				)
-			)
-		)
-		(property "LCSC Part" "C2170999"
-			(at 175.26 50.8 90)
-			(hide yes)
-			(show_name no)

Commit message: Asigning footprints for the ics
Parts:
- U3: footprint (none) -> Package_SO:SOIC-14_3.9x8.7mm_P1.27mm; LCSC Part (none) -> C5145433
- U4, U5: footprint (none) -> Package_SO:TSSOP-16_4.4x5mm_P0.65mm; LCSC Part (none) -> C2862976
Changed lines of the file:
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@@
 			)
 		)
-		(property "Footprint" ""
+		(property "Footprint" "Package_SO:SOIC-14_3.9x8.7mm_P1.27mm"
 			(at 218.44 63.5 0)
 			(hide yes)
@@
 		)
 		(property "Description" "Quad And 2 inputs"
+			(at 218.44 63.5 0)
+			(hide yes)
+			(show_name no)
+			(do_not_autoplace no)
+			(effects
+				(font
+					(size 1.27 1.27)
+				)
+			)
+		)
+		(property "LCSC Part" "C5145433"
 			(at 218.44 63.5 0)
 			(hide yes)
@@
 			)
 		)
-		(property "Footprint" ""
+		(property "Footprint" "Package_SO:TSSOP-16_4.4x5mm_P0.65mm"
 			(at 179.07 71.12 0)
 			(hide yes)
@@
 		)
 		(property "Description" "4 bits programmable counter"
+			(at 179.07 71.12 0)
+			(hide yes)
+			(show_name no)
+			(do_not_autoplace no)
+			(effects
+				(font
+					(size 1.27 1.27)
+				)
+			)
+		)
+		(property "LCSC Part" "C2862976"
 			(at 179.07 71.12 0)
 			(hide yes)
@@
 			)
 		)
-		(property "Footprint" ""
+		(property "Footprint" "Package_SO:TSSOP-16_4.4x5mm_P0.65mm"
 			(at 85.09 80.01 0)
 			(hide yes)
@@
 		)
 		(property "Description" "4 bits programmable counter"
+			(at 85.09 80.01 0)
+			(hide yes)
+			(show_name no)
+			(do_not_autoplace no)
+			(effects
+				(font
+					(size 1.27 1.27)
+				)
+			)
+		)
+		(property "LCSC Part" "C2862976"
 			(at 85.09 80.01 0)
 			(hide yes)
@@
 			)
 		)
-		(property "Footprint" ""
+		(property "Footprint" "Package_SO:SOIC-14_3.9x8.7mm_P1.27mm"
 			(at 124.46 74.93 0)
 			(hide yes)
@@
 		)
 		(property "Description" "Quad And 2 inputs"
+			(at 124.46 74.93 0)
+			(hide yes)
+			(show_name no)
+			(do_not_autoplace no)
+			(effects
+				(font
+					(size 1.27 1.27)
+				)
+			)
+		)
+		(property "LCSC Part" "C5145433"
 			(at 124.46 74.93 0)
 			(hide yes)
@@
 			)
 		)
-		(property "Footprint" ""
+		(property "Footprint" "Package_SO:SOIC-14_3.9x8.7mm_P1.27mm"
 			(at 50.8 173.99 0)
 			(hide yes)
@@
 			(at 50.8 173.99 0)
 			(hide yes)
+			(show_name no)
+			(do_not_autoplace no)
+			(effects
+				(font
+					(size 1.27 1.27)
+				)
+			)
+		)
+		(property "LCSC Part" "C5145433"
+			(at 50.8 173.99 0)
+			(hide yes)
