File: sec.kicad_sch (KiCad schematic)
At the start: 6 parts, among them U3 4081, U4 4510, U5 4510

Commit message: finishing the footprint asigment
Parts:
- C5, C6, C7: footprint (none) -> Resistor_SMD:R_0603_1608Metric; LCSC Part (none) -> C1591
- U3: footprint (none) -> Package_SO:SOIC-14_3.9x8.7mm_P1.27mm; LCSC Part (none) -> C40551
- U3: footprint Package_DIP:DIP-14_W7.62mm_Socket_LongPads -> Package_SO:SOIC-14_3.9x8.7mm_P1.27mm; LCSC Part (none) -> C40551
- U4, U5: footprint (none) -> Package_SO:TSSOP-16_4.4x5mm_P0.65mm; LCSC Part (none) -> C2862976
Changed lines of the file:
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@@
 			)
 		)
-		(property "Footprint" ""
+		(property "Footprint" "Resistor_SMD:R_0603_1608Metric"
 			(at 85.09 58.7248 0)
 			(hide yes)
@@
 			)
 		)
+		(property "LCSC Part" "C1591"
+			(at 81.28 59.69 90)
+			(hide yes)
+			(show_name no)
+			(do_not_autoplace no)
+			(effects
+				(font
+					(size 1.27 1.27)
+				)
+			)
+		)
 		(pin "1"
 		)
@@
 			)
 		)
-		(property "Footprint" ""
+		(property "Footprint" "Resistor_SMD:R_0603_1608Metric"
 			(at 50.8 157.7848 0)
 			(hide yes)
@@
 		(property "Description" "Unpolarized capacitor"
 			(at 46.99 158.75 0)
+			(hide yes)
+			(show_name no)
+			(do_not_autoplace no)
+			(effects
+				(font
+					(size 1.27 1.27)
+				)
+			)
+		)
+		(property "LCSC Part" "C1591"
+			(at 46.99 158.75 90)
 			(hide yes)
 			(show_name no)
@@
 			)
 		)
-		(property "Footprint" ""
+		(property "Footprint" "Package_SO:SOIC-14_3.9x8.7mm_P1.27mm"
 			(at 218.44 63.5 0)
 			(hide yes)
@@
 			)
 		)
+		(property "LCSC Part" "C40551"
+			(at 218.44 63.5 0)
+			(hide yes)
+			(show_name no)
+			(do_not_autoplace no)
+			(effects
+				(font
+					(size 1.27 1.27)
+				)
+			)
+		)
 		(pin "4"
 		)
@@
 			)
 		)
-		(property "Footprint" ""
+		(property "Footprint" "Package_SO:TSSOP-16_4.4x5mm_P0.65mm"
 			(at 179.07 71.12 0)
 			(hide yes)
@@
 			)
 		)
+		(property "LCSC Part" "C2862976"
+			(at 179.07 71.12 0)
+			(hide yes)
+			(show_name no)
+			(do_not_autoplace no)
+			(effects
+				(font
+					(size 1.27 1.27)
+				)
+			)
+		)
 		(pin "12"
 		)
@@
 			)
 		)
-		(property "Footprint" ""
+		(property "Footprint" "Package_SO:TSSOP-16_4.4x5mm_P0.65mm"
 			(at 85.09 80.01 0)
 			(hide yes)
@@
 			)
 		)
+		(property "LCSC Part" "C2862976"
+			(at 85.09 80.01 0)
+			(hide yes)
+			(show_name no)
+			(do_not_autoplace no)
+			(effects
+				(font
+					(size 1.27 1.27)
+				)
+			)
+		)
 		(pin "12"
 		)
@@
 			)
 		)
-		(property "Footprint" "Package_DIP:DIP-14_W7.62mm_Socket_LongPads"
+		(property "Footprint" "Package_SO:SOIC-14_3.9x8.7mm_P1.27mm"
 			(at 124.46 74.93 0)
 			(hide yes)
@@
 		)
 		(property "Description" "Quad And 2 inputs"
+			(at 124.46 74.93 0)
+			(hide yes)
+			(show_name no)
+			(do_not_autoplace no)
+			(effects
+				(font
+					(size 1.27 1.27)
+				)
+			)
+		)
+		(property "LCSC Part" "C40551"
 			(at 124.46 74.93 0)
 			(hide yes)
@@
 			)
 		)
-		(property "Footprint" ""
+		(property "Footprint" "Package_SO:SOIC-14_3.9x8.7mm_P1.27mm"
 			(at 50.8 173.99 0)
 			(hide yes)
@@
 			)
 		)
+		(property "LCSC Part" "C40551"
+			(at 50.8 173.99 0)
+			(hide yes)
+			(show_name no)
+			(do_not_autoplace no)
+			(effects
+				(font
+					(size 1.27 1.27)
+				)
+			)
+		)
 		(pin "4"
 		)
@@
 			)
 		)
-		(property "Footprint" ""
+		(property "Footprint" "Resistor_SMD:R_0603_1608Metric"
 			(at 179.07 49.8348 0)
 			(hide yes)
@@
 			(hide yes)
 			(show_name no)
+			(do_not_autoplace no)
+			(effects
+				(font
+					(size 1.27 1.27)
+				)
+			)
+		)
+		(property "LCSC Part" "C1591"
+			(at 175.26 50.8 90)
+			(hide yes)
+			(show_name no)
