File: clk.kicad_sch (KiCad schematic)
At the start: 9 parts, among them U1 4060, U2 4013, Y1 32.768 kHz

Commit message: finishing the footprint asigment
Parts:
- C1, C2: footprint (none) -> Resistor_SMD:R_0603_1608Metric; LCSC Part (none) -> C326840
- C3, C4: footprint (none) -> Resistor_SMD:R_0603_1608Metric; LCSC Part (none) -> C1591
- R1: footprint (none) -> Resistor_SMD:R_0603_1608Metric; LCSC Part (none) -> C2907027
- R2: footprint (none) -> Resistor_SMD:R_0603_1608Metric; LCSC Part (none) -> C2930145
- U1: footprint (none) -> Package_SO:SOIC-16_3.9x9.9mm_P1.27mm; LCSC Part (none) -> C134017
- U2: footprint (none) -> Package_SO:SOIC-14_3.9x8.7mm_P1.27mm; LCSC Part (none) -> C13527
- Y1: footprint (none) -> Crystal:Crystal_C38-LF_D3.0mm_L8.0mm_Horizontal; LCSC Part (none) -> C3034396
Changed lines of the file:
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@@
 			)
 		)
-		(property "Footprint" ""
+		(property "Footprint" "Package_SO:SOIC-14_3.9x8.7mm_P1.27mm"
 			(at 200.66 67.31 0)
 			(hide yes)
@@
 		)
 		(property "Description" "Dual D  FlipFlop, Set & reset"
+			(at 200.66 67.31 0)
+			(hide yes)
+			(show_name no)
+			(do_not_autoplace no)
+			(effects
+				(font
+					(size 1.27 1.27)
+				)
+			)
+		)
+		(property "LCSC Part" "C13527"
 			(at 200.66 67.31 0)
 			(hide yes)
@@
 			)
 		)
-		(property "Footprint" ""
+		(property "Footprint" "Package_SO:SOIC-14_3.9x8.7mm_P1.27mm"
 			(at 156.21 96.52 0)
 			(hide yes)
@@
 		)
 		(property "Description" "Dual D  FlipFlop, Set & reset"
+			(at 156.21 96.52 0)
+			(hide yes)
+			(show_name no)
+			(do_not_autoplace no)
+			(effects
+				(font
+					(size 1.27 1.27)
+				)
+			)
+		)
+		(property "LCSC Part" "C13527"
 			(at 156.21 96.52 0)
 			(hide yes)
@@
 			)
 		)
-		(property "Footprint" ""
+		(property "Footprint" "Resistor_SMD:R_0603_1608Metric"
 			(at 78.74 72.898 90)
 			(hide yes)
@@
 		(property "Description" "Resistor"
 			(at 78.74 71.12 0)
+			(hide yes)
+			(show_name no)
+			(do_not_autoplace no)
+			(effects
+				(font
+					(size 1.27 1.27)
+				)
+			)
+		)
+		(property "LCSC Part" "C2907027"
+			(at 78.74 71.12 90)
 			(hide yes)
 			(show_name no)
@@
 			)
 		)
-		(property "Footprint" ""
+		(property "Footprint" "Package_SO:SOIC-16_3.9x9.9mm_P1.27mm"
 			(at 115.57 86.36 0)
 			(hide yes)
@@
 			)
 		)
+		(property "LCSC Part" "C134017"
+			(at 115.57 83.82 0)
+			(hide yes)
+			(show_name no)
+			(do_not_autoplace no)
+			(effects
+				(font
+					(size 1.27 1.27)
+				)
+			)
+		)
 		(pin "3"
 		)
@@
 			)
 		)
-		(property "Footprint" ""
+		(property "Footprint" "Resistor_SMD:R_0603_1608Metric"
 			(at 62.23 64.4652 0)
 			(hide yes)
@@
 		(property "Description" "Unpolarized capacitor"
 			(at 66.04 63.5 0)
+			(hide yes)
+			(show_name no)
+			(do_not_autoplace no)
+			(effects
+				(font
+					(size 1.27 1.27)
+				)
+			)
+		)
+		(property "LCSC Part" "C326840"
+			(at 66.04 63.5 90)
 			(hide yes)
 			(show_name no)
@@
 			)
 		)
-		(property "Footprint" ""
+		(property "Footprint" "Resistor_SMD:R_0603_1608Metric"
 			(at 84.582 74.93 90)
 			(hide yes)
@@
 			)
 		)
+		(property "LCSC Part" "C2930145"
+			(at 86.36 74.93 0)
+			(hide yes)
+			(show_name no)
+			(do_not_autoplace no)
+			(effects
+				(font
+					(size 1.27 1.27)
+				)
+			)
+		)
 		(pin "2"
 		)
@@
 			)
 		)
-		(property "Footprint" ""
+		(property "Footprint" "Resistor_SMD:R_0603_1608Metric"
 			(at 62.23 83.5152 0)
 			(hide yes)
@@
 		(property "Description" "Unpolarized capacitor"
 			(at 66.04 82.55 0)
+			(hide yes)
+			(show_name no)
+			(do_not_autoplace no)
+			(effects
+				(font
+					(size 1.27 1.27)
+				)
+			)
+		)
+		(property "LCSC Part" "C326840"
+			(at 66.04 82.55 90)
 			(hide yes)
 			(show_name no)
@@
 			)
 		)
-		(property "Footprint" ""
+		(property "Footprint" "Crystal:Crystal_C38-LF_D3.0mm_L8.0mm_Horizontal"
 			(at 69.85 74.93 0)
 			(hide yes)
@@
 		(property "Description" "Two pin crystal"
 			(at 69.85 74.93 0)
+			(hide yes)
+			(show_name no)
+			(do_not_autoplace no)
+			(effects
+				(font
+					(size 1.27 1.27)
+				)
+			)
+		)
+		(property "LCSC Part" "C3034396"
+			(at 69.85 74.93 90)
 			(hide yes)
 			(show_name no)
@@
 			)
 		)
-		(property "Footprint" ""
+		(property "Footprint" "Resistor_SMD:R_0603_1608Metric"
 			(at 152.4 123.4948 0)
 			(hide yes)
@@
 		(property "Description" "Unpolarized capacitor"
 			(at 148.59 124.46 0)
+			(hide yes)
+			(show_name no)
+			(do_not_autoplace no)
+			(effects
+				(font
+					(size 1.27 1.27)
+				)
+			)
+		)
+		(property "LCSC Part" "C1591"
+			(at 148.59 124.46 90)
 			(hide yes)
 			(show_name no)
@@
 			)
 		)
-		(property "Footprint" ""
+		(property "Footprint" "Resistor_SMD:R_0603_1608Metric"
 			(at 115.57 59.9948 0)
 			(hide yes)
@@
 		(property "Description" "Unpolarized capacitor"
 			(at 111.76 60.96 0)
+			(hide yes)
+			(show_name no)
+			(do_not_autoplace no)
+			(effects
+				(font
+					(size 1.27 1.27)
+				)
+			)
+		)
+		(property "LCSC Part" "C1591"
+			(at 111.76 60.96 90)
 			(hide yes)
 			(show_name no)
@@
 			)
 		)
-		(property "Footprint" ""
+		(property "Footprint" "Package_SO:SOIC-14_3.9x8.7mm_P1.27mm"
 			(at 152.4 139.7 0)
 			(hide yes)
@@
 			(at 152.4 139.7 0)
 			(hide yes)
+			(show_name no)
+			(do_not_autoplace no)
+			(effects
+				(font
+					(size 1.27 1.27)
+				)
+			)
+		)
+		(property "LCSC Part" "C13527"
+			(at 152.4 139.7 0)
+			(hide yes)

Commit message: start to make the clk signal
Connections:
- net at C1.1, R1.1: now also Y1.1; no longer Y1.2
- net at C2.1, R2.2, U1.11 (~{Φ1}): now also Y1.2; no longer Y1.1
Other:
- moved on the sheet: Y1
Changed lines of the file:
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@@
+	)
+	(junction
+		(at 69.85 78.74)
+		(diameter 0)
+		(color 0 0 0 0)
+	)
+	(junction
+		(at 152.4 124.46)
+		(diameter 0)
+		(color 0 0 0 0)
 	)
 	(junction
@@
 	)
 	(junction
-		(at 152.4 124.46)
-		(diameter 0)
-		(color 0 0 0 0)
-	)
-	(junction
 		(at 86.36 71.12)
-		(diameter 0)
-		(color 0 0 0 0)
-	)
-	(junction
-		(at 69.85 78.74)
 		(diameter 0)
 		(color 0 0 0 0)
@@
 	(symbol
 		(lib_id "Device:Crystal")
-		(at 69.85 74.93 90)
+		(at 69.85 74.93 270)
 		(unit 1)
 		(body_style 1)
@@
 		(dnp no)
 		(property "Reference" "Y1"
-			(at 61.087 73.025 90)
+			(at 78.613 76.835 90)
 			(show_name no)
 			(do_not_autoplace no)
@@
 		)
 		(property "Value" "32.768 kHz"
-			(at 61.087 75.565 90)
-			(show_name no)
-			(do_not_autoplace no)
+			(at 78.613 74.295 90)
+			(show_name no)
+			(do_not_autoplace no)

Commit message: designing the layout and duing the routing
Parts:
- renumbered C3 to C1, C1 to C2, C2 to C3, U2 to U1, U1 to U2
Changed lines of the file:
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@@
 		(in_pos_files yes)
 		(dnp no)
-		(property "Reference" "#PWR02"
+		(property "Reference" "#PWR09"
 			(at 55.88 82.55 0)
 			(hide yes)
@@
 			(project "BinaryClock"
 				(path "/b8db7867-2c41-4996-89b7-85623a375f4b/06cc8139-062b-489e-8e2f-c0ae5744b4b6"
-					(reference "#PWR02")
+					(reference "#PWR09")
 					(unit 1)
 				)
@@
 		(in_pos_files yes)
 		(dnp no)
-		(property "Reference" "#PWR01"
+		(property "Reference" "#PWR04"
 			(at 55.88 63.5 0)
 			(hide yes)
@@
 			(project "BinaryClock"
 				(path "/b8db7867-2c41-4996-89b7-85623a375f4b/06cc8139-062b-489e-8e2f-c0ae5744b4b6"
-					(reference "#PWR01")
+					(reference "#PWR04")
 					(unit 1)
 				)
@@
 		(dnp no)
 		(fields_autoplaced yes)
-		(property "Reference" "#PWR07"
+		(property "Reference" "#PWR014"
 			(at 138.43 124.46 0)
 			(hide yes)
@@
 			(project "BinaryClock"
 				(path "/b8db7867-2c41-4996-89b7-85623a375f4b/06cc8139-062b-489e-8e2f-c0ae5744b4b6"
-					(reference "#PWR07")
+					(reference "#PWR014")
 					(unit 1)
 				)
@@
 		(dnp no)
 		(fields_autoplaced yes)
-		(property "Reference" "#PWR04"
+		(property "Reference" "#PWR03"
 			(at 101.6 60.96 0)
 			(hide yes)
@@
 			(project "BinaryClock"
 				(path "/b8db7867-2c41-4996-89b7-85623a375f4b/06cc8139-062b-489e-8e2f-c0ae5744b4b6"
-					(reference "#PWR04")
+					(reference "#PWR03")
 					(unit 1)
 				)
@@
 		(dnp no)
 		(fields_autoplaced yes)
-		(property "Reference" "#PWR015"
+		(property "Reference" "#PWR07"
 			(at 200.66 81.28 0)
 			(hide yes)
@@
 			(project "BinaryClock"
 				(path "/b8db7867-2c41-4996-89b7-85623a375f4b/06cc8139-062b-489e-8e2f-c0ae5744b4b6"
-					(reference "#PWR015")
+					(reference "#PWR07")
 					(unit 1)
 				)
@@
 		(dnp no)
 		(fields_autoplaced yes)
-		(property "Reference" "U2"
+		(property "Reference" "U1"
 			(at 202.8033 57.15 0)
 			(show_name no)
@@
 			(project "BinaryClock"
 				(path "/b8db7867-2c41-4996-89b7-85623a375f4b/06cc8139-062b-489e-8e2f-c0ae5744b4b6"
-					(reference "U2")
+					(reference "U1")
 					(unit 2)
 				)
@@
 		(dnp no)
 		(fields_autoplaced yes)
-		(property "Reference" "U2"
+		(property "Reference" "U1"
 			(at 158.3533 86.36 0)
 			(show_name no)
@@
 			(project "BinaryClock"
 				(path "/b8db7867-2c41-4996-89b7-85623a375f4b/06cc8139-062b-489e-8e2f-c0ae5744b4b6"
-					(reference "U2")
+					(reference "U1")
 					(unit 1)
 				)
@@
 		(in_pos_files yes)
 		(dnp no)
-		(property "Reference" "#PWR011"
+		(property "Reference" "#PWR012"
 			(at 156.21 110.49 0)
 			(hide yes)
@@
 			(project "BinaryClock"
 				(path "/b8db7867-2c41-4996-89b7-85623a375f4b/06cc8139-062b-489e-8e2f-c0ae5744b4b6"
-					(reference "#PWR011")
+					(reference "#PWR012")
 					(unit 1)
 				)
@@
 		(dnp no)
 		(fields_autoplaced yes)
-		(property "Reference" "U1"
+		(property "Reference" "U2"
 			(at 117.7133 63.5 0)
 			(show_name no)
@@
 			(project "BinaryClock"
 				(path "/b8db7867-2c41-4996-89b7-85623a375f4b/06cc8139-062b-489e-8e2f-c0ae5744b4b6"
-					(reference "U1")
+					(reference "U2")
 					(unit 1)
 				)
@@
 		(in_pos_files yes)
 		(dnp no)
-		(property "Reference" "C1"
+		(property "Reference" "C2"
 			(at 64.135 69.469 90)
 			(show_name no)
@@
 			(project "BinaryClock"
 				(path "/b8db7867-2c41-4996-89b7-85623a375f4b/06cc8139-062b-489e-8e2f-c0ae5744b4b6"
-					(reference "C1")
+					(reference "C2")
 					(unit 1)
 				)
@@
 		(dnp no)
 		(fields_autoplaced yes)
-		(property "Reference" "#PWR012"
+		(property "Reference" "#PWR05"
 			(at 186.69 64.77 0)
 			(hide yes)
@@
 			(project "BinaryClock"
 				(path "/b8db7867-2c41-4996-89b7-85623a375f4b/06cc8139-062b-489e-8e2f-c0ae5744b4b6"
-					(reference "#PWR012")
+					(reference "#PWR05")
 					(unit 1)
 				)
@@
 		(in_pos_files yes)
 		(dnp no)
-		(property "Reference" "C2"
+		(property "Reference" "C3"
 			(at 67.437 90.0429 90)
 			(show_name no)
@@
 			(project "BinaryClock"
 				(path "/b8db7867-2c41-4996-89b7-85623a375f4b/06cc8139-062b-489e-8e2f-c0ae5744b4b6"
-					(reference "C2")
+					(reference "C3")
 					(unit 1)
 				)
@@
 		(dnp no)
 		(fields_autoplaced yes)
-		(property "Reference" "#PWR08"
+		(property "Reference" "#PWR013"
 			(at 152.4 125.73 0)
 			(hide yes)
@@
 			(project "BinaryClock"
 				(path "/b8db7867-2c41-4996-89b7-85623a375f4b/06cc8139-062b-489e-8e2f-c0ae5744b4b6"
-					(reference "#PWR08")
+					(reference "#PWR013")
 					(unit 1)
 				)
@@
 		(dnp no)
 		(fields_autoplaced yes)
-		(property "Reference" "#PWR09"
+		(property "Reference" "#PWR015"
 			(at 152.4 156.21 0)
 			(hide yes)
@@
 			(project "BinaryClock"
 				(path "/b8db7867-2c41-4996-89b7-85623a375f4b/06cc8139-062b-489e-8e2f-c0ae5744b4b6"
-					(reference "#PWR09")
+					(reference "#PWR015")
 					(unit 1)
 				)
@@
 		(dnp no)
 		(fields_autoplaced yes)
-		(property "Reference" "#PWR014"
+		(property "Reference" "#PWR02"
 			(at 200.66 53.34 0)
 			(hide yes)
@@
 			(project "BinaryClock"
 				(path "/b8db7867-2c41-4996-89b7-85623a375f4b/06cc8139-062b-489e-8e2f-c0ae5744b4b6"
-					(reference "#PWR014")
+					(reference "#PWR02")
 					(unit 1)
 				)
@@
 		(dnp no)
 		(fields_autoplaced yes)
-		(property "Reference" "#PWR03"
+		(property "Reference" "#PWR08"
 			(at 96.52 81.28 0)
 			(hide yes)
@@
 			(project "BinaryClock"
 				(path "/b8db7867-2c41-4996-89b7-85623a375f4b/06cc8139-062b-489e-8e2f-c0ae5744b4b6"
-					(reference "#PWR03")
+					(reference "#PWR08")
 					(unit 1)
 				)
@@
 		(dnp no)
 		(fields_autoplaced yes)
-		(property "Reference" "#PWR05"
+		(property "Reference" "#PWR01"
 			(at 115.57 62.23 0)
 			(hide yes)
@@
 			(project "BinaryClock"
 				(path "/b8db7867-2c41-4996-89b7-85623a375f4b/06cc8139-062b-489e-8e2f-c0ae5744b4b6"
-					(reference "#PWR05")
+					(reference "#PWR01")
 					(unit 1)
 				)
@@
 		(in_pos_files yes)
 		(dnp no)
-		(property "Reference" "C3"
+		(property "Reference" "C1"
 			(at 111.76 57.658 90)
 			(show_name no)
@@
 			(project "BinaryClock"
 				(path "/b8db7867-2c41-4996-89b7-85623a375f4b/06cc8139-062b-489e-8e2f-c0ae5744b4b6"
-					(reference "C3")
+					(reference "C1")
 					(unit 1)
 				)
@@
 		(dnp no)
 		(fields_autoplaced yes)
-		(property "Reference" "#PWR013"
+		(property "Reference" "#PWR06"
 			(at 186.69 67.31 0)
 			(hide yes)
@@
 			(project "BinaryClock"
 				(path "/b8db7867-2c41-4996-89b7-85623a375f4b/06cc8139-062b-489e-8e2f-c0ae5744b4b6"
-					(reference "#PWR013")
+					(reference "#PWR06")
 					(unit 1)
 				)
@@
 		(dnp no)
 		(fields_autoplaced yes)
-		(property "Reference" "U2"
+		(property "Reference" "U1"
 			(at 158.75 138.4299 0)
 			(show_name no)
@@
 			(project "BinaryClock"
 				(path "/b8db7867-2c41-4996-89b7-85623a375f4b/06cc8139-062b-489e-8e2f-c0ae5744b4b6"
-					(reference "U2")
+					(reference "U1")
 					(unit 3)
 				)
@@
 		(dnp no)
 		(fields_autoplaced yes)
-		(property "Reference" "#PWR06"
+		(property "Reference" "#PWR011"
 			(at 115.57 110.49 0)
 			(hide yes)
@@
 			(project "BinaryClock"
 				(path "/b8db7867-2c41-4996-89b7-85623a375f4b/06cc8139-062b-489e-8e2f-c0ae5744b4b6"
-					(reference "#PWR06")
+					(reference "#PWR011")
 					(unit 1)
 				)
