File: power.kicad_sch (KiCad schematic)
At the start: 5 parts, among them U12 HX TYPE-C 6PIN

Commit message: Asigning footprints for the ics
Parts:
- C18: LCSC Part (none) -> C88726
Changed lines of the file:
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@@
+			)
+		)
+		(property "LCSC Part" "C88726"
+			(at 93.98 104.14 90)
+			(hide yes)
+			(show_name no)
+			(do_not_autoplace no)
+			(effects
+				(font
+					(size 1.27 1.27)
+				)
 			)
 		)
