File: power.kicad_sch (KiCad schematic)
At the start: 0 parts

Commit message: Designing the base circuit of the usb-c
Parts:
- added C18: 75uF, symbol Device:C_Polarized
- added C19: 100nf, symbol Device:C
- added R11, R12: 5.1k, symbol Device:R
- added U12: HX TYPE-C 6PIN, EasyEDA:USB-C-SMD_HX-TYPE-C-6PIN, symbol EasyEDA:HXTYPE-C6PIN
Connections:
- new net: R11.2, U12.A5 (CC1)
- new net: R12.1, U12.B5 (CC2)
- new net +5V: C18.1, C19.1, U12.A9 (VBUS), U12.B9 (VBUS)
- new net GND: C18.2, C19.2, R11.1, R12.2, U12.13 (EH), U12.14 (EH), U12.15 (EH), U12.16 (EH), U12.A12 (GND), U12.B12 (GND)

Commit message: finished the power input
Parts:
- C18: value 75uF -> 10uF
Changed lines of the file:
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@@
 			)
 		)
-		(property "Value" "75uF"
+		(property "Value" "10uF"
 			(at 93.091 99.06 90)
 			(show_name no)

Commit message: finishing the footprint asigment
Parts:
- C18: footprint (none) -> Capacitor_SMD:CP_Elec_6.3x7.7; LCSC Part (none) -> C72478
- C19: value 100nf -> 100nF; footprint (none) -> Resistor_SMD:R_0603_1608Metric; LCSC Part (none) -> C1591
- R11, R12: footprint (none) -> Resistor_SMD:R_0603_1608Metric; LCSC Part (none) -> C2907044
Changed lines of the file:
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@@
 			)
 		)
-		(property "Footprint" ""
+		(property "Footprint" "Resistor_SMD:R_0603_1608Metric"
 			(at 101.6 83.058 90)
 			(hide yes)
@@
 		(property "Description" "Resistor"
 			(at 101.6 81.28 0)
+			(hide yes)
+			(show_name no)
+			(do_not_autoplace no)
+			(effects
+				(font
+					(size 1.27 1.27)
+				)
+			)
+		)
+		(property "LCSC Part" "C2907044"
+			(at 101.6 81.28 90)
 			(hide yes)
 			(show_name no)
@@
 			)
 		)
-		(property "Footprint" ""
+		(property "Footprint" "Capacitor_SMD:CP_Elec_6.3x7.7"
 			(at 97.79 103.1748 0)
 			(hide yes)
@@
 		(property "Description" "Polarized capacitor"
 			(at 93.98 104.14 0)
+			(hide yes)
+			(show_name no)
+			(do_not_autoplace no)
+			(effects
+				(font
+					(size 1.27 1.27)
+				)
+			)
+		)
+		(property "LCSC Part" "C72478"
+			(at 93.98 104.14 90)
 			(hide yes)
 			(show_name no)
@@
 			)
 		)
-		(property "Footprint" ""
+		(property "Footprint" "Resistor_SMD:R_0603_1608Metric"
 			(at 71.12 83.058 90)
 			(hide yes)
@@
 		(property "Description" "Resistor"
 			(at 71.12 81.28 0)
+			(hide yes)
+			(show_name no)
+			(do_not_autoplace no)
+			(effects
+				(font
+					(size 1.27 1.27)
+				)
+			)
+		)
+		(property "LCSC Part" "C2907044"
+			(at 71.12 81.28 90)
 			(hide yes)
 			(show_name no)
@@
 			)
 		)
-		(property "Value" "100nf"
+		(property "Value" "100nF"
 			(at 93.98 110.744 90)
 			(show_name no)
@@
 			)
 		)
-		(property "Footprint" ""
+		(property "Footprint" "Resistor_SMD:R_0603_1608Metric"
 			(at 97.79 113.3348 0)
 			(hide yes)
@@
 			(hide yes)
 			(show_name no)
+			(do_not_autoplace no)
+			(effects
+				(font
+					(size 1.27 1.27)
+				)
+			)
+		)
+		(property "LCSC Part" "C1591"
+			(at 93.98 114.3 90)
+			(hide yes)
+			(show_name no)

Commit message: starting the layout
Parts:
- removed U12: HX TYPE-C 6PIN, EasyEDA:USB-C-SMD_HX-TYPE-C-6PIN, symbol EasyEDA:HXTYPE-C6PIN
- added J1: USB_C_Receptacle_PowerOnly_6P, Connector_USB:USB_C_Receptacle_GCT_USB4105-xx-A_16P_TopMnt_Horizontal, symbol Connector:USB_C_Receptacle_PowerOnly_6P
Connections:
- net +5V: now also J1.A9 (VBUS), J1.B9 (VBUS)
- net GND: now also J1.A12 (GND), J1.B12 (GND), J1.SH (SHIELD)
- net at R11.2: now also J1.A5 (CC1)
- net at R12.1: now also J1.B5 (CC2)

Commit message: start to make the clk signal
Parts:
- J1: footprint Connector_USB:USB_C_Receptacle_GCT_USB4105-xx-A_16P_TopMnt_Horizontal -> Connector_USB:USB_C_Receptacle_GCT_USB4125-xx-x-0190_6P_TopMnt_Horizontal
Changed lines of the file:
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@@
 			)
 		)
-		(property "Footprint" "Connector_USB:USB_C_Receptacle_GCT_USB4105-xx-A_16P_TopMnt_Horizontal"
+		(property "Footprint" "Connector_USB:USB_C_Receptacle_GCT_USB4125-xx-x-0190_6P_TopMnt_Horizontal"
 			(at 43.18 95.25 0)
 			(hide yes)
