File: hour.kicad_sch (KiCad schematic)
At the start: 15 parts, among them SW3 SW_MEC_5G, SW7 SW_Push_Dual, U10 4081, U11 4510, U6 4071, U9 4510

Commit message: designing the layout and duing the routing
Parts:
- removed SW3: SW_MEC_5G, Button_Switch_THT:SW_PUSH_6mm_H5mm, symbol Switch:SW_MEC_5G
- added SW4: SW_Push_Dual, Button_Switch_THT:SW_PUSH_6mm_H5mm, symbol Switch:SW_Push_Dual
- renumbered C15 to C13, C17 to C14, C14 to C15, C13 to C16, C16 to C17, R7 to R10, R10 to R7, R9 to R8, R8 to R9, SW7 to SW3, U9 to U11, U6 to U7, U11 to U9
Connections:
- net +5V: now also SW4.1
- net at R10.1, R9.1: now also SW4.2
