File: min.kicad_sch (KiCad schematic)
At the start: 15 parts, among them SW1 SW_MEC_5G, SW2 SW_MEC_5G, U3 4081, U6 4071, U7 4510, U8 4510

Commit message: starting the layout
Parts:
- removed SW1, SW2: SW_MEC_5G, Button_Switch_THT:SW_PUSH_6mm_H5mm, symbol Switch:SW_MEC_5G
- added SW5, SW6: SW_Push_Dual, Button_Switch_THT:SW_PUSH_6mm_H5mm, symbol Switch:SW_Push_Dual
Connections:
- net +5V: now also SW5.1, SW6.1
- net at R3.1, R4.1: now also SW5.2
- net at R5.1, R6.1: now also SW6.2

Commit message: designing the layout and duing the routing
Parts:
- renumbered C8 to C11, C9 to C12, C11 to C8, C12 to C9, R6 to R3, R5 to R4, R4 to R5, R3 to R6, SW6 to SW1, SW5 to SW2, U8 to U6, U6 to U7, U7 to U8
