File: sec_display.kicad_sch (KiCad schematic)
At the start: 5 parts

Commit message: Asigning footprints
Parts:
- removed RN1: R_Pack04_SIP, Resistor_THT:R_Array_SIP8, symbol Device:R_Pack04_SIP
- added RN1: 4D03WGJ0102T5E, EasyEDA:RES-ARRAY-SMD_0603-8P-L3.2-W1.6-BL, symbol EasyEDA:4D03WGJ0102T5E
- D1, D2, D3, D4: footprint (none) -> LED_THT:LED_D3.0mm; LCSC Part (none) -> C779430
Connections:
- net 1: now also RN1.1
- net 2: now also RN1.2
- net 4: now also RN1.3
- net 8: now also RN1.4
- net at D2.1 (K): now also RN1.6
- net at D4.1 (K): now also RN1.5
- net at D1.1 (K): now also RN1.8
- net at D3.1 (K): now also RN1.7

Commit message: Asigning footprints
Parts:
- removed RN1: 4D03WGJ0102T5E, EasyEDA:RES-ARRAY-SMD_0603-8P-L3.2-W1.6-BL, symbol EasyEDA:4D03WGJ0102T5E
- added RN1: R_Pack04_SIP, Resistor_THT:R_Array_SIP8, symbol Device:R_Pack04_SIP
- D1, D2, D3, D4: footprint LED_THT:LED_D3.0mm -> LED_THT:LED_D3.0mm_Clear; LCSC Part C779430 -> (none)
Connections:
- net 1: now also RN1.1 (R1.1)
- net 2: now also RN1.3 (R2.1)
- net 4: now also RN1.5 (R3.1)
- net 8: now also RN1.7 (R4.1)
- net at D2.1 (K): now also RN1.6 (R3.2)
- net at D4.1 (K): now also RN1.8 (R4.2)
- net at D3.1 (K): now also RN1.4 (R2.2)
- net at D1.1 (K): now also RN1.2 (R1.2)

Commit message: Asigning footprints for the ics
Parts:
- RN1: footprint Resistor_THT:R_Array_SIP8 -> EasyEDA:RES-ARRAY-SMD_0603-8P-L3.2-W1.6-BL; LCSC Part (none) -> C20197
Changed lines of the file:
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@@
 			)
 		)
-		(property "Footprint" "Resistor_THT:R_Array_SIP8"
+		(property "Footprint" "EasyEDA:RES-ARRAY-SMD_0603-8P-L3.2-W1.6-BL"
 			(at 81.28 118.745 90)
 			(hide yes)
@@
 			(hide yes)
 			(show_name no)
+			(do_not_autoplace no)
+			(effects
+				(font
+					(size 1.27 1.27)
+				)
+			)
+		)
+		(property "LCSC Part" "C20197"
+			(at 81.28 101.6 90)
+			(hide yes)
+			(show_name no)
