File: sec_display.kicad_sch (KiCad schematic)
At the start: 5 parts

Commit message: finishing the footprint asigment
Parts:
- D1, D2, D3, D4: footprint (none) -> LED_SMD:LED_1206_3216Metric; LCSC Part (none) -> C375482
- RN1: LCSC Part (none) -> C12018
Changed lines of the file:
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@@
 			)
 		)
-		(property "Footprint" ""
+		(property "Footprint" "LED_SMD:LED_1206_3216Metric"
 			(at 67.31 106.68 0)
 			(hide yes)
@@
 		)
 		(property "Sim.Pins" "1=K 2=A"
+			(at 67.31 106.68 0)
+			(hide yes)
+			(show_name no)
+			(do_not_autoplace no)
+			(effects
+				(font
+					(size 1.27 1.27)
+				)
+			)
+		)
+		(property "LCSC Part" "C375482"
 			(at 67.31 106.68 0)
 			(hide yes)
@@
 			)
 		)
-		(property "Footprint" ""
+		(property "Footprint" "LED_SMD:LED_1206_3216Metric"
 			(at 72.39 114.3 0)
 			(hide yes)
@@
 		)
 		(property "Sim.Pins" "1=K 2=A"
+			(at 72.39 114.3 0)
+			(hide yes)
+			(show_name no)
+			(do_not_autoplace no)
+			(effects
+				(font
+					(size 1.27 1.27)
+				)
+			)
+		)
+		(property "LCSC Part" "C375482"
 			(at 72.39 114.3 0)
 			(hide yes)
@@
 			)
 		)
+		(property "LCSC Part" "C12018"
+			(at 81.28 101.6 90)
+			(hide yes)
+			(show_name no)
+			(do_not_autoplace no)
+			(effects
+				(font
+					(size 1.27 1.27)
+				)
+			)
+		)
 		(pin "2"
 		)
@@
 			)
 		)
-		(property "Footprint" ""
+		(property "Footprint" "LED_SMD:LED_1206_3216Metric"
 			(at 67.31 91.44 0)
 			(hide yes)
@@
 		)
 		(property "Sim.Pins" "1=K 2=A"
+			(at 67.31 91.44 0)
+			(hide yes)
+			(show_name no)
+			(do_not_autoplace no)
+			(effects
+				(font
+					(size 1.27 1.27)
+				)
+			)
+		)
+		(property "LCSC Part" "C375482"
 			(at 67.31 91.44 0)
 			(hide yes)
@@
 			)
 		)
-		(property "Footprint" ""
+		(property "Footprint" "LED_SMD:LED_1206_3216Metric"
 			(at 72.39 99.06 0)
 			(hide yes)
@@
 			(at 72.39 99.06 0)
 			(hide yes)
+			(show_name no)
+			(do_not_autoplace no)
+			(effects
+				(font
+					(size 1.27 1.27)
+				)
+			)
+		)
+		(property "LCSC Part" "C375482"
+			(at 72.39 99.06 0)
+			(hide yes)

Commit message: start to make the clk signal
Parts:
- RN1: footprint Resistor_THT:R_Array_SIP8 -> Resistor_SMD:R_Array_Convex_4x1206
Changed lines of the file:
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@@
 			)
 		)
-		(property "Footprint" "Resistor_THT:R_Array_SIP8"
+		(property "Footprint" "Resistor_SMD:R_Array_Convex_4x1206"
 			(at 81.28 118.745 90)
 			(hide yes)

Commit message: designing the layout and duing the routing
Parts:
- renumbered D3 to D2, D2 to D3
Changed lines of the file:
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@@
 		(in_pos_files yes)
 		(dnp no)
-		(property "Reference" "D2"
+		(property "Reference" "D3"
 			(at 68.834 110.998 0)
 			(show_name no)
@@
 			(project "BinaryClock"
 				(path "/b8db7867-2c41-4996-89b7-85623a375f4b/d72dbc43-5f9c-4389-b46b-bcc9f20f0691/72c2d78a-d678-45bf-be56-716a4bf4e93c"
-					(reference "D10")
+					(reference "D11")
 					(unit 1)
 				)
 				(path "/b8db7867-2c41-4996-89b7-85623a375f4b/d72dbc43-5f9c-4389-b46b-bcc9f20f0691/8a27fff0-1362-4f1a-9796-2225af35d845"
-					(reference "D22")
+					(reference "D23")
 					(unit 1)
 				)
 				(path "/b8db7867-2c41-4996-89b7-85623a375f4b/d72dbc43-5f9c-4389-b46b-bcc9f20f0691/9d667165-1e46-420a-b7c2-c853bd88335e"
-					(reference "D14")
+					(reference "D15")
 					(unit 1)
 				)
 				(path "/b8db7867-2c41-4996-89b7-85623a375f4b/d72dbc43-5f9c-4389-b46b-bcc9f20f0691/a2fc0f23-edba-4a42-809e-31a5704900ef"
-					(reference "D6")
+					(reference "D7")
 					(unit 1)
 				)
 				(path "/b8db7867-2c41-4996-89b7-85623a375f4b/d72dbc43-5f9c-4389-b46b-bcc9f20f0691/c511b7b7-1902-4f18-9b6d-bdf563bc0fbd"
-					(reference "D2")
+					(reference "D3")
 					(unit 1)
 				)
 				(path "/b8db7867-2c41-4996-89b7-85623a375f4b/d72dbc43-5f9c-4389-b46b-bcc9f20f0691/ca0ecceb-e5a9-4cc1-9364-faafc2408685"
-					(reference "D18")
+					(reference "D19")
 					(unit 1)
 				)
@@
 		(dnp no)
 		(fields_autoplaced yes)
-		(property "Reference" "#PWR0116"
+		(property "Reference" "#PWR0111"
 			(at 62.23 99.06 0)
 			(hide yes)
@@
 			(project "BinaryClock"
 				(path "/b8db7867-2c41-4996-89b7-85623a375f4b/d72dbc43-5f9c-4389-b46b-bcc9f20f0691/72c2d78a-d678-45bf-be56-716a4bf4e93c"
-					(reference "#PWR0124")
+					(reference "#PWR0119")
 					(unit 1)
 				)
 				(path "/b8db7867-2c41-4996-89b7-85623a375f4b/d72dbc43-5f9c-4389-b46b-bcc9f20f0691/8a27fff0-1362-4f1a-9796-2225af35d845"
-					(reference "#PWR0136")
+					(reference "#PWR0131")
 					(unit 1)
 				)
 				(path "/b8db7867-2c41-4996-89b7-85623a375f4b/d72dbc43-5f9c-4389-b46b-bcc9f20f0691/9d667165-1e46-420a-b7c2-c853bd88335e"
-					(reference "#PWR0128")
+					(reference "#PWR0123")
 					(unit 1)
 				)
 				(path "/b8db7867-2c41-4996-89b7-85623a375f4b/d72dbc43-5f9c-4389-b46b-bcc9f20f0691/a2fc0f23-edba-4a42-809e-31a5704900ef"
-					(reference "#PWR0120")
+					(reference "#PWR0115")
 					(unit 1)
 				)
 				(path "/b8db7867-2c41-4996-89b7-85623a375f4b/d72dbc43-5f9c-4389-b46b-bcc9f20f0691/c511b7b7-1902-4f18-9b6d-bdf563bc0fbd"
-					(reference "#PWR0116")
+					(reference "#PWR0111")
 					(unit 1)
 				)
 				(path "/b8db7867-2c41-4996-89b7-85623a375f4b/d72dbc43-5f9c-4389-b46b-bcc9f20f0691/ca0ecceb-e5a9-4cc1-9364-faafc2408685"
-					(reference "#PWR0132")
+					(reference "#PWR0127")
 					(unit 1)
 				)
@@
 		(dnp no)
 		(fields_autoplaced yes)
-		(property "Reference" "#PWR0114"
+		(property "Reference" "#PWR0110"
 			(at 57.15 91.44 0)
 			(hide yes)
@@
 			(project "BinaryClock"
 				(path "/b8db7867-2c41-4996-89b7-85623a375f4b/d72dbc43-5f9c-4389-b46b-bcc9f20f0691/72c2d78a-d678-45bf-be56-716a4bf4e93c"
+					(reference "#PWR0118")
+					(unit 1)
+				)
+				(path "/b8db7867-2c41-4996-89b7-85623a375f4b/d72dbc43-5f9c-4389-b46b-bcc9f20f0691/8a27fff0-1362-4f1a-9796-2225af35d845"
+					(reference "#PWR0130")
+					(unit 1)
+				)
+				(path "/b8db7867-2c41-4996-89b7-85623a375f4b/d72dbc43-5f9c-4389-b46b-bcc9f20f0691/9d667165-1e46-420a-b7c2-c853bd88335e"
 					(reference "#PWR0122")
 					(unit 1)
 				)
-				(path "/b8db7867-2c41-4996-89b7-85623a375f4b/d72dbc43-5f9c-4389-b46b-bcc9f20f0691/8a27fff0-1362-4f1a-9796-2225af35d845"
-					(reference "#PWR0134")
-					(unit 1)
-				)
-				(path "/b8db7867-2c41-4996-89b7-85623a375f4b/d72dbc43-5f9c-4389-b46b-bcc9f20f0691/9d667165-1e46-420a-b7c2-c853bd88335e"
+				(path "/b8db7867-2c41-4996-89b7-85623a375f4b/d72dbc43-5f9c-4389-b46b-bcc9f20f0691/a2fc0f23-edba-4a42-809e-31a5704900ef"
+					(reference "#PWR0114")
+					(unit 1)
+				)
+				(path "/b8db7867-2c41-4996-89b7-85623a375f4b/d72dbc43-5f9c-4389-b46b-bcc9f20f0691/c511b7b7-1902-4f18-9b6d-bdf563bc0fbd"
+					(reference "#PWR0110")
+					(unit 1)
+				)
+				(path "/b8db7867-2c41-4996-89b7-85623a375f4b/d72dbc43-5f9c-4389-b46b-bcc9f20f0691/ca0ecceb-e5a9-4cc1-9364-faafc2408685"
 					(reference "#PWR0126")
-					(unit 1)
-				)
-				(path "/b8db7867-2c41-4996-89b7-85623a375f4b/d72dbc43-5f9c-4389-b46b-bcc9f20f0691/a2fc0f23-edba-4a42-809e-31a5704900ef"
-					(reference "#PWR0118")
-					(unit 1)
-				)
-				(path "/b8db7867-2c41-4996-89b7-85623a375f4b/d72dbc43-5f9c-4389-b46b-bcc9f20f0691/c511b7b7-1902-4f18-9b6d-bdf563bc0fbd"
-					(reference "#PWR0114")
-					(unit 1)
-				)
-				(path "/b8db7867-2c41-4996-89b7-85623a375f4b/d72dbc43-5f9c-4389-b46b-bcc9f20f0691/ca0ecceb-e5a9-4cc1-9364-faafc2408685"
-					(reference "#PWR0130")
 					(unit 1)
 				)
@@
 		(dnp no)
 		(fields_autoplaced yes)
-		(property "Reference" "#PWR0117"
+		(property "Reference" "#PWR0113"
 			(at 62.23 114.3 0)
 			(hide yes)
@@
 			(project "BinaryClock"
 				(path "/b8db7867-2c41-4996-89b7-85623a375f4b/d72dbc43-5f9c-4389-b46b-bcc9f20f0691/72c2d78a-d678-45bf-be56-716a4bf4e93c"
+					(reference "#PWR0121")
+					(unit 1)
+				)
+				(path "/b8db7867-2c41-4996-89b7-85623a375f4b/d72dbc43-5f9c-4389-b46b-bcc9f20f0691/8a27fff0-1362-4f1a-9796-2225af35d845"
+					(reference "#PWR0133")
+					(unit 1)
+				)
+				(path "/b8db7867-2c41-4996-89b7-85623a375f4b/d72dbc43-5f9c-4389-b46b-bcc9f20f0691/9d667165-1e46-420a-b7c2-c853bd88335e"
 					(reference "#PWR0125")
 					(unit 1)
 				)
-				(path "/b8db7867-2c41-4996-89b7-85623a375f4b/d72dbc43-5f9c-4389-b46b-bcc9f20f0691/8a27fff0-1362-4f1a-9796-2225af35d845"
-					(reference "#PWR0137")
-					(unit 1)
-				)
-				(path "/b8db7867-2c41-4996-89b7-85623a375f4b/d72dbc43-5f9c-4389-b46b-bcc9f20f0691/9d667165-1e46-420a-b7c2-c853bd88335e"
+				(path "/b8db7867-2c41-4996-89b7-85623a375f4b/d72dbc43-5f9c-4389-b46b-bcc9f20f0691/a2fc0f23-edba-4a42-809e-31a5704900ef"
+					(reference "#PWR0117")
+					(unit 1)
+				)
+				(path "/b8db7867-2c41-4996-89b7-85623a375f4b/d72dbc43-5f9c-4389-b46b-bcc9f20f0691/c511b7b7-1902-4f18-9b6d-bdf563bc0fbd"
+					(reference "#PWR0113")
+					(unit 1)
+				)
+				(path "/b8db7867-2c41-4996-89b7-85623a375f4b/d72dbc43-5f9c-4389-b46b-bcc9f20f0691/ca0ecceb-e5a9-4cc1-9364-faafc2408685"
 					(reference "#PWR0129")
-					(unit 1)
-				)
-				(path "/b8db7867-2c41-4996-89b7-85623a375f4b/d72dbc43-5f9c-4389-b46b-bcc9f20f0691/a2fc0f23-edba-4a42-809e-31a5704900ef"
-					(reference "#PWR0121")
-					(unit 1)
-				)
-				(path "/b8db7867-2c41-4996-89b7-85623a375f4b/d72dbc43-5f9c-4389-b46b-bcc9f20f0691/c511b7b7-1902-4f18-9b6d-bdf563bc0fbd"
-					(reference "#PWR0117")
-					(unit 1)
-				)
-				(path "/b8db7867-2c41-4996-89b7-85623a375f4b/d72dbc43-5f9c-4389-b46b-bcc9f20f0691/ca0ecceb-e5a9-4cc1-9364-faafc2408685"
-					(reference "#PWR0133")
 					(unit 1)
 				)
@@
 		(dnp no)
 		(fields_autoplaced yes)
-		(property "Reference" "#PWR0115"
+		(property "Reference" "#PWR0112"
 			(at 57.15 106.68 0)
 			(hide yes)
@@
 			(project "BinaryClock"
 				(path "/b8db7867-2c41-4996-89b7-85623a375f4b/d72dbc43-5f9c-4389-b46b-bcc9f20f0691/72c2d78a-d678-45bf-be56-716a4bf4e93c"
-					(reference "#PWR0123")
+					(reference "#PWR0120")
 					(unit 1)
 				)
 				(path "/b8db7867-2c41-4996-89b7-85623a375f4b/d72dbc43-5f9c-4389-b46b-bcc9f20f0691/8a27fff0-1362-4f1a-9796-2225af35d845"
-					(reference "#PWR0135")
+					(reference "#PWR0132")
 					(unit 1)
 				)
 				(path "/b8db7867-2c41-4996-89b7-85623a375f4b/d72dbc43-5f9c-4389-b46b-bcc9f20f0691/9d667165-1e46-420a-b7c2-c853bd88335e"
-					(reference "#PWR0127")
+					(reference "#PWR0124")
 					(unit 1)
 				)
 				(path "/b8db7867-2c41-4996-89b7-85623a375f4b/d72dbc43-5f9c-4389-b46b-bcc9f20f0691/a2fc0f23-edba-4a42-809e-31a5704900ef"
-					(reference "#PWR0119")
+					(reference "#PWR0116")
 					(unit 1)
 				)
 				(path "/b8db7867-2c41-4996-89b7-85623a375f4b/d72dbc43-5f9c-4389-b46b-bcc9f20f0691/c511b7b7-1902-4f18-9b6d-bdf563bc0fbd"
-					(reference "#PWR0115")
+					(reference "#PWR0112")
 					(unit 1)
 				)
 				(path "/b8db7867-2c41-4996-89b7-85623a375f4b/d72dbc43-5f9c-4389-b46b-bcc9f20f0691/ca0ecceb-e5a9-4cc1-9364-faafc2408685"
-					(reference "#PWR0131")
+					(reference "#PWR0128")
 					(unit 1)
 				)
@@
 		(in_pos_files yes)
 		(dnp no)
-		(property "Reference" "D3"
+		(property "Reference" "D2"
 			(at 72.136 103.632 0)
 			(show_name no)
@@
 			(project "BinaryClock"
 				(path "/b8db7867-2c41-4996-89b7-85623a375f4b/d72dbc43-5f9c-4389-b46b-bcc9f20f0691/72c2d78a-d678-45bf-be56-716a4bf4e93c"
-					(reference "D11")
+					(reference "D10")
 					(unit 1)
 				)
 				(path "/b8db7867-2c41-4996-89b7-85623a375f4b/d72dbc43-5f9c-4389-b46b-bcc9f20f0691/8a27fff0-1362-4f1a-9796-2225af35d845"
-					(reference "D23")
+					(reference "D22")
 					(unit 1)
 				)
 				(path "/b8db7867-2c41-4996-89b7-85623a375f4b/d72dbc43-5f9c-4389-b46b-bcc9f20f0691/9d667165-1e46-420a-b7c2-c853bd88335e"
-					(reference "D15")
+					(reference "D14")
 					(unit 1)
 				)
 				(path "/b8db7867-2c41-4996-89b7-85623a375f4b/d72dbc43-5f9c-4389-b46b-bcc9f20f0691/a2fc0f23-edba-4a42-809e-31a5704900ef"
-					(reference "D7")
+					(reference "D6")
 					(unit 1)
 				)
 				(path "/b8db7867-2c41-4996-89b7-85623a375f4b/d72dbc43-5f9c-4389-b46b-bcc9f20f0691/c511b7b7-1902-4f18-9b6d-bdf563bc0fbd"
-					(reference "D3")
+					(reference "D2")
 					(unit 1)
 				)
 				(path "/b8db7867-2c41-4996-89b7-85623a375f4b/d72dbc43-5f9c-4389-b46b-bcc9f20f0691/ca0ecceb-e5a9-4cc1-9364-faafc2408685"
-					(reference "D19")
-					(unit 1)
-				)
+					(reference "D18")
+					(unit 1)
+				)
