File: BinaryClock.kicad_pcb (KiCad board)
At the start: 2 copper layers, 79 parts, among them J1 USB_C_Receptacle_PowerOnly_6P, SW2 SW_MEC_5G, SW3 SW_MEC_5G, SW4 SW_MEC_5G, SW5 SW_Push_Dual, U1 4060, U10 4081, U11 4510, U2 4013, U3 4081, U4 4510, U5 4510, U6 4071, U7 4510, U8 4510, U9 4510, Y1 32.768 kHz

Commit message: start to make the clk signal
Parts:
- removed SW2, SW4: SW_MEC_5G, Button_Switch_THT:SW_PUSH_6mm_H5mm
- removed the SW5 at (14.1, 43.3)
- removed the SW5 at (28.8, 28.8)
- added SW5: SW_Push_Dual, Button_Switch_THT:SW_PUSH_6mm_H5mm, F.Cu at (24.6, 20.1)
- added SW6: SW_Push_Dual, Button_Switch_THT:SW_PUSH_6mm_H5mm, F.Cu at (24.6, 28.7)
- added SW7: SW_Push_Dual, Button_Switch_THT:SW_PUSH_6mm_H5mm, F.Cu at (50.3, 28.7)
- J1: footprint Connector_USB:USB_C_Receptacle_GCT_USB4105-xx-A_16P_TopMnt_Horizontal -> Connector_USB:USB_C_Receptacle_GCT_USB4125-xx-x-0190_6P_TopMnt_Horizontal
- RN1, RN2, RN3, RN4, RN5, RN6: footprint Resistor_THT:R_Array_SIP8 -> Resistor_SMD:R_Array_Convex_4x1206
- moved C4 160.8 mm to (137.9, 166.7)
- moved RN1 141.9 mm to (144.5, 185.7)
- moved D2 134.0 mm to (139.0, 187.4)
- moved D4 134.0 mm to (139.0, 194.2)
- moved D1 134.0 mm to (139.0, 184.0)
- moved D3 134.0 mm to (139.0, 190.8)
- moved C1 124.1 mm to (144.5, 77.5), turned to -90 degrees
- moved C2 121.8 mm to (144.5, 70.0), turned to 90 degrees
- moved Y1 119.7 mm to (144.5, 74.7), turned to 90 degrees
- moved R1 119.1 mm to (142.2, 74.5), turned to 180 degrees
- moved J1 117.7 mm to (167.4, 102.2), turned to 90 degrees
- moved R2 115.6 mm to (139.2, 73.8), turned to 90 degrees
- moved C3 115.6 mm to (139.1, 67.0), turned to 180 degrees
- moved R11 102.3 mm to (159.9, 103.3)
- moved C18 100.8 mm to (154.5, 99.4), turned to 90 degrees
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Connections:
- Y1 pad 1: Net-(U1-~{Φ1}) -> Net-(C1-Pad1)
- Y1 pad 2: Net-(C1-Pad1) -> Net-(U1-~{Φ1})
Routing:
- net +5V: track 0.00 -> 88.1 mm
- net GND: track 0.00 -> 27.1 mm, vias 0 -> 15
- net Net-(U1-Q14): track 0.00 -> 17.2 mm
- net Net-(U1-~{Φ1}): track 0.00 -> 10.6 mm
- net Net-(U2A-D): track 0.00 -> 7.50 mm
- net Net-(U1-Φ0): track 0.00 -> 6.25 mm
- net Net-(C1-Pad1): track 0.00 -> 3.48 mm
- added copper zone on B.Cu, net GND

Commit message: designing the layout and duing the routing
Parts:
- removed the SW3 at (50.3, 20.1)
- added SW4: SW_Push_Dual, Button_Switch_THT:SW_PUSH_6mm_H5mm, F.Cu at (105.9, 60.6)
- moved RN1 140.8 mm to (68.1, 67.4), turned to 180 degrees
- moved C4 132.8 mm to (134.8, 33.9), turned to 90 degrees
- moved D2 129.2 mm to (78.1, 76.9)
- moved D1 128.5 mm to (68.1, 76.9)
- moved D4 124.3 mm to (98.1, 76.9)
- moved D3 121.7 mm to (88.1, 76.9)
- moved U8 108.3 mm to (113.9, 22.1)
- moved U7 100.7 mm to (99.5, 39.4)
- moved C8 80.8 mm to (98.5, 48.0), turned to 180 degrees
- moved R4 79.0 mm to (98.5, 49.6), turned to 180 degrees
- moved R3 78.8 mm to (98.5, 51.2), turned to 180 degrees
- moved SW1 78.1 mm to (95.9, 60.6), turned to 90 degrees
- moved C9 76.5 mm to (96.8, 23.5)
- moved C7 76.4 mm to (121.4, 28.9)
- moved C13 76.1 mm to (118.5, 48.0), turned to 180 degrees
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- renumbered C3 to C1, C8 to C11, C9 to C12, C15 to C13, C17 to C14, C14 to C15, C13 to C16, C16 to C17, C1 to C2, C2 to C3, C7 to C5, C5 to C7, C11 to C8, C12 to C9, D11 to D10, D10 to D11, D15 to D14, D14 to D15, D19 to D18, D18 to D19, D3 to D2, D23 to D22, D22 to D23, D2 to D3, D7 to D6, D6 to D7, R7 to R10, R6 to R3, R5 to R4, R4 to R5, R3 to R6, R10 to R7, R9 to R8, R8 to R9, SW6 to SW1, SW5 to SW2, SW7 to SW3, U2 to U1, U9 to U11, U1 to U2, U5 to U4, U4 to U5, U8 to U6, U6 to U7, U7 to U8, U11 to U9
Routing:
- net +5V: track 88.1 -> 356.1 mm, vias 0 -> 12
- net GND: track 27.1 -> 162.0 mm, vias 15 -> 114
- net /Counters/hour/24h_RST: track 0.00 -> 129.0 mm, vias 0 -> 2
- net /Counters/min/min-o_1: track 0.00 -> 117.0 mm, vias 0 -> 2
- net /Counters/min/min-o_4: track 0.00 -> 112.8 mm, vias 0 -> 4
- net /Counters/hour/hour-t_4: track 0.00 -> 100.2 mm, vias 0 -> 2
- net /Counters/hour/hour-t_1: track 0.00 -> 96.7 mm, vias 0 -> 4
- net /Counters/min/min-t_3: track 0.00 -> 93.3 mm, vias 0 -> 6
- net /Counters/min/min-o_3: track 0.00 -> 91.3 mm, vias 0 -> 2
- net /Counters/sec/sec-o_3: track 0.00 -> 88.8 mm, vias 0 -> 2
- net /Counters/hour/hour-t_3: track 0.00 -> 85.8 mm, vias 0 -> 2
- net /Counters/sec/sec-o_2: track 0.00 -> 79.5 mm, vias 0 -> 3
- net /Counters/min/min-o_2: track 0.00 -> 78.5 mm, vias 0 -> 2
- net /Counters/sec/sec-t_4: track 0.00 -> 77.0 mm, vias 0 -> 4
- net /Counters/hour/hour-t_2: track 0.00 -> 76.1 mm, vias 0 -> 4
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