File: pcb/BinaryClock.kicad_pcb (KiCad board)
At the start: 2 copper layers, 78 parts, among them J1 USB_C_Receptacle_PowerOnly_6P, SW1 SW_Push_Dual, SW2 SW_Push_Dual, SW3 SW_Push_Dual, SW4 SW_Push_Dual, U1 4013, U10 4081, U11 4510, U2 4060, U3 4081, U4 4510, U5 4510, U6 4510, U7 4071, U8 4510, U9 4510, Y1 32.768 kHz

Commit message: organising
Routing:
- net +5V: track 356.1 -> 363.8 mm, vias 12 -> 13
Other:
- board outline added: 98.3 x 80.3 mm
Changed lines of the file:
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@@
 		)
 	)
+	(gr_rect
+		(start 57 15.7)
+		(end 155.3 96)
+		(stroke
+			(width 0.05)
+			(type default)
+		)
+		(fill no)
+		(layer "Edge.Cuts")
+	)
 	(segment
 		(start 100.2952 62.588)
@@
 	)
 	(segment
+		(start 116.725 23.675)
+		(end 119.475 23.675)
+		(width 0.5)
+		(layer "F.Cu")
+		(net "+5V")
+	)
+	(segment
 		(start 80.9125 23.5)
 		(end 80.9125 24.2125)
@@
 	)
 	(segment
+		(start 119.5 23.7)
+		(end 119.475 23.675)
+		(width 0.5)
+		(layer "F.Cu")
+		(net "+5V")
+	)
+	(segment
 		(start 123.2 28.9)
 		(end 123.3 28.8)
@@
 	)
 	(via
+		(at 119.475 23.675)
+		(size 0.6)
+		(drill 0.3)
+		(layers "F.Cu" "B.Cu")
+		(net "+5V")
+	)
+	(via
 		(at 99 23.5)
 		(size 0.6)
@@
 	)
 	(segment
+		(start 124.075 23.675)
+		(end 124.3 23.9)
+		(width 0.5)
+		(layer "B.Cu")
+		(net "+5V")
+	)
+	(segment
 		(start 85.9 60.55)
 		(end 85.9 54.05)
@@
 		(width 0.5)
 		(layer "B.Cu")
+		(net "+5V")
+	)
+	(segment
+		(start 119.475 23.675)
+		(end 124.075 23.675)
+		(width 0.5)
+		(layer "B.Cu")

Commit message: generating the produstion files
Parts:
- added REF**: MountingHole_2.2mm_M2, MountingHole:MountingHole_2.2mm_M2, F.Cu at (59.4, 101.7)
Other:
- board size 98.3 x 80.3 mm -> 98.3 x 89.3 mm
Changed lines of the file:
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@@
 		)
 	)
+	(footprint "MountingHole:MountingHole_2.2mm_M2"
+		(layer "F.Cu")
+		(at 59.4 101.7)
+		(descr "Mounting Hole 2.2mm, M2, no annular, generated by kicad-footprint-generator mountinghole.py")
+		(tags "mountinghole M2")
+		(property "Reference" "REF**"
+			(at 0 -3.15 0)
+			(layer "F.SilkS")
+			(effects
+				(font
+					(size 1 1)
+					(thickness 0.15)
+				)
+			)
+		)
+		(property "Value" "MountingHole_2.2mm_M2"
+			(at 0 3.15 0)
+			(layer "F.Fab")
+			(effects
+				(font
+					(size 1 1)
+					(thickness 0.15)
+				)
+			)
+		)
+		(property "Datasheet" ""
+			(at 0 0 0)
+			(layer "F.Fab")
+			(hide yes)
+			(effects
+				(font
+					(size 1.27 1.27)
+				)
+			)
+		)
+		(property "Description" ""
+			(at 0 0 0)
+			(layer "F.Fab")
+			(hide yes)
+			(effects
+				(font
+					(size 1.27 1.27)
+				)
+			)
+		)
+		(property "KiLib_Generator" "mounting_hardware/mounting_hole"
+			(at 0 0 0)
+			(layer "F.SilkS")
+			(hide yes)
+			(effects
+				(font
+					(size 1 1)
+					(thickness 0.15)
+				)
+			)
+		)
+		(attr exclude_from_pos_files exclude_from_bom)
+		(duplicate_pad_numbers_are_jumpers no)
+		(fp_circle
+			(center 0 0)
+			(end 2.2 0)
+			(stroke
+				(width 0.15)
+				(type solid)
+			)
+			(fill no)
+			(layer "Cmts.User")
+		)
+		(fp_circle
+			(center 0 0)
+			(end 2.45 0)
+			(stroke
+				(width 0.05)
+				(type solid)
+			)
+			(fill no)
+			(layer "F.CrtYd")
+		)
+		(fp_text user "${REFERENCE}"
+			(at 0 0 0)
+			(layer "F.Fab")
+			(effects
+				(font
+					(size 1 1)
+					(thickness 0.15)
+				)
+			)
+		)
+		(pad "" np_thru_hole circle
+			(at 0 0)
+			(size 2.2 2.2)
+			(drill 2.2)
+			(layers "*.Cu" "*.Mask")
+		)
+		(embedded_fonts no)
+	)
 	(footprint "Resistor_SMD:R_0603_1608Metric"
 		(layer "F.Cu")
@@
 	)
 	(gr_rect
-		(start 57 15.7)
-		(end 155.3 96)
+		(start 56.95 14.85)
+		(end 155.25 104.15)
 		(stroke
 			(width 0.05)
